File: MacroBoard/MacroBoard.kicad_pcb (KiCad board)
At the start: 2 copper layers, 103.3 x 105.9 mm, 106 parts, among them J1 TYPE-C-31-M12_13, SW1 SW_Push, SW2 RotaryEncoder_Switch, SW3 RotaryEncoder_Switch, U1 AT90USB1286-AU, U2 TPD4E05U06DQAR, Y1 Crystal_GND24_Small

Commit message: cleanup
Parts:
- added H1: MountingHole, MountingHole:MountingHole_2.2mm_M2, F.Cu at (130.0, 33.0)
- added H2: MountingHole, MountingHole:MountingHole_2.2mm_M2, F.Cu at (70.0, 90.6)
- added H3: MountingHole, MountingHole:MountingHole_2.2mm_M2, F.Cu at (168.0, 33.0)
- added H4: MountingHole, MountingHole:MountingHole_2.2mm_M2, F.Cu at (70.4, 33.0)
- added H5: MountingHole, MountingHole:MountingHole_2.2mm_M2, F.Cu at (168.0, 133.2)
- added H6: MountingHole, MountingHole:MountingHole_2.2mm_M2, F.Cu at (70.4, 133.2)
- added H7: MountingHole, MountingHole:MountingHole_2.2mm_M2, F.Cu at (119.2, 133.2)
- added H8: MountingHole, MountingHole:MountingHole_2.2mm_M2, F.Cu at (129.2, 95.4)
- added H9: MountingHole, MountingHole:MountingHole_2.2mm_M2, F.Cu at (168.2, 90.6)
- added R7: 60, Resistor_SMD:R_0402_1005Metric_Pad0.72x0.64mm_HandSolder, B.Cu at (84.2, 39.9)
- moved Y1 4.62 mm to (161.4, 34.2)
- moved C5 4.62 mm to (162.5, 37.6)
- moved C6 4.62 mm to (158.0, 33.1)
- moved D41 1.80 mm to (87.4, 46.5), turned to -90 degrees
- moved C1 1.00 mm to (85.6, 41.8)
- moved F1 1.00 mm to (84.6, 44.9)
Connections:
- D41 pad 2: VCC -> +5V
- F1 pad 2: VCC -> +5V
- J1 pad A4: VBUS -> Net-(J1-PadA4)
- J1 pad B4: VBUS -> Net-(J1-PadA4)
Routing:
- net +5V: track 451.2 -> 558.5 mm, vias 0 -> 5
- net GNDPWR: track 0.00 -> 17.0 mm
- net Net-(J1-PadA4): track 0.00 -> 8.78 mm
- net Net-(C5-Pad1): track 69.1 -> 64.2 mm
- net VCC: track 2.57 -> 0.00 mm
- net /ROT_2B: track 44.4 -> 42.7 mm
- net ROW2: track 206.2 -> 207.7 mm
- net ROW3: track 225.6 -> 227.2 mm
- net VBUS: track 5.60 -> 4.19 mm
- net /ROT_2A: track 40.6 -> 39.2 mm

Commit message: minor changes
Parts:
- moved SW2 1.15 mm to (138.1, 43.7)
- moved H9 0.91 mm to (168.3, 89.7)
- moved H4 0.71 mm to (69.8, 32.5)
- moved H6 0.57 mm to (69.8, 133.3)
- moved H3 0.53 mm to (168.3, 32.5)
- moved H5 0.31 mm to (168.3, 133.3)
- moved H2 0.19 mm to (69.8, 90.5)
- moved H7 0.15 mm to (119.2, 133.3)
Routing:
- net /ROT_1B: track 15.3 -> 16.4 mm
- net /ROT_1A: track 14.1 -> 15.3 mm
- net Net-(SW2-PadS2): track 27.5 -> 26.4 mm
- net ROW0: track 177.2 -> 176.7 mm
Other:
- board size 103.3 x 105.9 mm -> 103.5 x 105.8 mm

Commit message: generate final Gerber
Parts:
- added Q1: 2N7002, Package_TO_SOT_SMD:SOT-23, B.Cu at (72.4, 47.5)
- added R10: 46, Resistor_SMD:R_0805_2012Metric, B.Cu at (74.2, 50.6)
- added R8: 10k, Resistor_SMD:R_0805_2012Metric, B.Cu at (79.0, 50.5)
- added R9: 10k, Resistor_SMD:R_0805_2012Metric, B.Cu at (79.0, 47.5)
- R7: footprint Resistor_SMD:R_0402_1005Metric_Pad0.72x0.64mm_HandSolder -> Resistor_SMD:R_0805_2012Metric_Pad1.20x1.40mm_HandSolder
- moved R7 8.60 mm to (91.5, 44.5), turned to 45 degrees
- moved F1 1.80 mm to (84.6, 46.7)
- moved SW1 1.20 mm to (132.1, 48.8)
- moved C1 1.10 mm to (85.6, 42.9)
Connections:
- C10 pad 1: +5V -> /Power_LED
- C11 pad 1: +5V -> /Power_LED
- C12 pad 1: +5V -> /Power_LED
- C13 pad 1: +5V -> /Power_LED
- C14 pad 1: +5V -> /Power_LED
- C15 pad 1: +5V -> /Power_LED
- C16 pad 1: +5V -> /Power_LED
- C17 pad 1: +5V -> /Power_LED
- C18 pad 1: +5V -> /Power_LED
- C19 pad 1: +5V -> /Power_LED
- C20 pad 1: +5V -> /Power_LED
- C21 pad 1: +5V -> /Power_LED
- C22 pad 1: +5V -> /Power_LED
- C23 pad 1: +5V -> /Power_LED
- C24 pad 1: +5V -> /Power_LED
- C25 pad 1: +5V -> /Power_LED
- C26 pad 1: +5V -> /Power_LED
- C27 pad 1: +5V -> /Power_LED
- C28 pad 1: +5V -> /Power_LED
- C9 pad 1: +5V -> /Power_LED
- D21 pad 4: +5V -> /Power_LED
- D22 pad 4: +5V -> /Power_LED
- D23 pad 4: +5V -> /Power_LED
- D24 pad 4: +5V -> /Power_LED
- D25 pad 4: +5V -> /Power_LED
- D26 pad 4: +5V -> /Power_LED
- D27 pad 4: +5V -> /Power_LED
- D28 pad 4: +5V -> /Power_LED
- D29 pad 4: +5V -> /Power_LED
- D30 pad 4: +5V -> /Power_LED
- D31 pad 4: +5V -> /Power_LED
- D32 pad 4: +5V -> /Power_LED
- D33 pad 4: +5V -> /Power_LED
- D34 pad 4: +5V -> /Power_LED
- D35 pad 4: +5V -> /Power_LED
- D36 pad 4: +5V -> /Power_LED
- D37 pad 4: +5V -> /Power_LED
- D38 pad 4: +5V -> /Power_LED
- D39 pad 4: +5V -> /Power_LED
- D40 pad 4: +5V -> /Power_LED
- D41 pad 2: +5V -> /Power
- F1 pad 2: +5V -> /Power
- J1 pad A4: Net-(J1-PadA4) -> VBUS
- J1 pad B4: Net-(J1-PadA4) -> VBUS
- R7 pad 1: Net-(J1-PadA4) -> /Power
- R7 pad 2: VBUS -> +5V
- U1 pad 42: unconnected-(U1-Pad42) -> Net-(U1-Pad42)
Routing:
- net +5V: track 558.5 -> 75.3 mm, vias 5 -> 0
- net /Power_LED: track 0.00 -> 478.3 mm, vias 0 -> 6
- net /Power: track 0.00 -> 25.7 mm, vias 0 -> 2
- net Net-(U1-Pad42): track 0.00 -> 24.9 mm
- net VBUS: track 4.19 -> 15.1 mm
- net Net-(J1-PadA4): track 8.78 -> 0.00 mm
- net Net-(Q1-Pad1): track 0.00 -> 8.13 mm
- net Net-(Q1-Pad2): track 0.00 -> 2.20 mm
- net GND: track 18.5 -> 19.7 mm
- net Net-(R6-Pad2): track 14.5 -> 15.8 mm

Commit message: fixed lights
Parts:
- D21, D22, D23, D24, D25, D26, D27, D28, D29, D30, D31, D32, D33, D34, D35, D36, D37, D38, D39, D40: footprint led:SK6812MINI_3.5x3.7mm_SMD-Flipped-Back -> led:SK6812MINI_3.4x3.0mm_SMD-Back-Flipped
- moved C20 12.1 mm to (124.9, 128.0), turned to 90 degrees
- moved C12 12.1 mm to (86.8, 128.0), turned to 90 degrees
- moved C14 12.0 mm to (105.7, 89.9), turned to 90 degrees
- moved C16 12.0 mm to (105.8, 128.0), turned to 90 degrees
- moved C24 12.0 mm to (143.9, 128.0), turned to 90 degrees
- moved C26 12.0 mm to (162.9, 89.9), turned to 90 degrees
- moved C28 12.0 mm to (162.9, 128.0), turned to 90 degrees
- moved C11 12.0 mm to (86.7, 109.0), turned to 90 degrees
- moved C23 12.0 mm to (143.9, 109.0), turned to 90 degrees
- moved C15 11.9 mm to (105.7, 108.9), turned to 90 degrees
- moved C22 11.9 mm to (143.8, 89.9), turned to 90 degrees
- moved C18 11.9 mm to (124.8, 89.9), turned to 90 degrees
- moved C17 11.9 mm to (124.7, 70.9), turned to 90 degrees
- moved C25 11.9 mm to (162.8, 70.9), turned to 90 degrees
- moved C27 11.9 mm to (162.9, 109.0), turned to 90 degrees
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Connections:
- D21 pad 1: Net-(D21-Pad1) -> /Power_LED
- D21 pad 2: GNDREF -> Net-(D21-Pad2)
- D21 pad 3: DataIN -> GNDREF
- D21 pad 4: /Power_LED -> DataIN
- D22 pad 1: Net-(D22-Pad1) -> /Power_LED
- D22 pad 2: GNDREF -> Net-(D22-Pad2)
- D22 pad 3: Net-(D22-Pad3) -> GNDREF
- D22 pad 4: /Power_LED -> Net-(D22-Pad4)
- D23 pad 1: Net-(D23-Pad1) -> /Power_LED
- D23 pad 2: GNDREF -> Net-(D23-Pad2)
- D23 pad 3: Net-(D23-Pad3) -> GNDREF
- D23 pad 4: /Power_LED -> Net-(D23-Pad4)
- D24 pad 1: Net-(D24-Pad1) -> /Power_LED
- D24 pad 2: GNDREF -> Net-(D24-Pad2)
- D24 pad 3: Net-(D24-Pad3) -> GNDREF
- D24 pad 4: /Power_LED -> Net-(D24-Pad4)
- D25 pad 1: Net-(D25-Pad1) -> /Power_LED
- D25 pad 2: GNDREF -> Net-(D25-Pad2)
- D25 pad 3: Net-(D21-Pad1) -> GNDREF
- D25 pad 4: /Power_LED -> Net-(D21-Pad2)
- D26 pad 1: Net-(D26-Pad1) -> /Power_LED
- D26 pad 2: GNDREF -> Net-(D26-Pad2)
- D26 pad 3: Net-(D22-Pad1) -> GNDREF
- D26 pad 4: /Power_LED -> Net-(D22-Pad2)
- D27 pad 1: Net-(D27-Pad1) -> /Power_LED
- D27 pad 2: GNDREF -> Net-(D27-Pad2)
- D27 pad 3: Net-(D23-Pad1) -> GNDREF
- D27 pad 4: /Power_LED -> Net-(D23-Pad2)
- D28 pad 1: Net-(D28-Pad1) -> /Power_LED
- D28 pad 2: GNDREF -> Net-(D28-Pad2)
- D28 pad 3: Net-(D24-Pad1) -> GNDREF
- D28 pad 4: /Power_LED -> Net-(D24-Pad2)
- D29 pad 1: Net-(D29-Pad1) -> /Power_LED
- D29 pad 2: GNDREF -> Net-(D29-Pad2)
- D29 pad 3: Net-(D25-Pad1) -> GNDREF
- D29 pad 4: /Power_LED -> Net-(D25-Pad2)
- D30 pad 1: Net-(D30-Pad1) -> /Power_LED
- D30 pad 2: GNDREF -> Net-(D30-Pad2)
- D30 pad 3: Net-(D26-Pad1) -> GNDREF
- D30 pad 4: /Power_LED -> Net-(D26-Pad2)
- D31 pad 1: Net-(D31-Pad1) -> /Power_LED
- D31 pad 2: GNDREF -> Net-(D31-Pad2)
- D31 pad 3: Net-(D27-Pad1) -> GNDREF
- D31 pad 4: /Power_LED -> Net-(D27-Pad2)
- D32 pad 1: Net-(D32-Pad1) -> /Power_LED
- D32 pad 2: GNDREF -> Net-(D32-Pad2)
- D32 pad 3: Net-(D28-Pad1) -> GNDREF
- D32 pad 4: /Power_LED -> Net-(D28-Pad2)
- D33 pad 1: Net-(D33-Pad1) -> /Power_LED
- D33 pad 2: GNDREF -> Net-(D33-Pad2)
- D33 pad 3: Net-(D29-Pad1) -> GNDREF
- D33 pad 4: /Power_LED -> Net-(D29-Pad2)
- D34 pad 1: Net-(D34-Pad1) -> /Power_LED
- D34 pad 2: GNDREF -> Net-(D34-Pad2)
- D34 pad 3: Net-(D30-Pad1) -> GNDREF
- D34 pad 4: /Power_LED -> Net-(D30-Pad2)
- D35 pad 1: Net-(D35-Pad1) -> /Power_LED
- D35 pad 2: GNDREF -> Net-(D35-Pad2)
- D35 pad 3: Net-(D31-Pad1) -> GNDREF
- D35 pad 4: /Power_LED -> Net-(D31-Pad2)
- D36 pad 1: Net-(D36-Pad1) -> /Power_LED
- D36 pad 2: GNDREF -> Net-(D36-Pad2)
- D36 pad 3: Net-(D32-Pad1) -> GNDREF
- D36 pad 4: /Power_LED -> Net-(D32-Pad2)
- D37 pad 1: Net-(D22-Pad3) -> /Power_LED
- D37 pad 2: GNDREF -> Net-(D22-Pad4)
- D37 pad 3: Net-(D33-Pad1) -> GNDREF
- D37 pad 4: /Power_LED -> Net-(D33-Pad2)
- D38 pad 1: Net-(D23-Pad3) -> /Power_LED
- D38 pad 2: GNDREF -> Net-(D23-Pad4)
- D38 pad 3: Net-(D34-Pad1) -> GNDREF
- D38 pad 4: /Power_LED -> Net-(D34-Pad2)
- D39 pad 1: Net-(D24-Pad3) -> /Power_LED
- D39 pad 2: GNDREF -> Net-(D24-Pad4)
- D39 pad 3: Net-(D35-Pad1) -> GNDREF
- D39 pad 4: /Power_LED -> Net-(D35-Pad2)
- D40 pad 1: DataOUT -> /Power_LED
- D40 pad 2: GNDREF -> DataOUT
- D40 pad 3: Net-(D36-Pad1) -> GNDREF
- D40 pad 4: /Power_LED -> Net-(D36-Pad2)
- SW2 pad S2: Net-(SW2-PadS2) -> COL5
- SW3 pad S2: Net-(SW2-PadS2) -> COL5
- U1 pad 11: unconnected-(U1-Pad11) -> /ROT_2A
- U1 pad 12: /ROT_2A -> /ROT_2B
- U1 pad 13: /ROT_2B -> COL5
- U1 pad 33: COL0 -> DataIN
- U1 pad 34: COL1 -> COL0
- U1 pad 35: COL2 -> COL1
- U1 pad 36: COL3 -> COL2
- U1 pad 37: COL4 -> COL3
- U1 pad 38: COL5 -> COL4
Routing:
- net Net-(D24-Pad4): track 0.00 -> 126.1 mm, vias 0 -> 2
- net Net-(D22-Pad4): track 0.00 -> 125.7 mm, vias 0 -> 2
- net Net-(D23-Pad4): track 0.00 -> 124.7 mm, vias 0 -> 2
- net Net-(D24-Pad3): track 111.9 -> 0.00 mm, vias 2 -> 0
- net Net-(D22-Pad3): track 111.7 -> 0.00 mm, vias 2 -> 0
- net Net-(D23-Pad3): track 111.6 -> 0.00 mm, vias 2 -> 0
- net DataIN: track 0.00 -> 59.6 mm
- net COL5: track 0.00 -> 59.4 mm, vias 0 -> 1
- net /Power_LED: track 478.3 -> 514.2 mm
- net Net-(SW2-PadS2): track 26.4 -> 0.00 mm
- net Net-(D24-Pad2): track 0.00 -> 14.8 mm
- net Net-(D32-Pad2): track 0.00 -> 14.8 mm
- net Net-(D30-Pad2): track 0.00 -> 14.8 mm
- net Net-(D26-Pad2): track 0.00 -> 14.8 mm
- net Net-(D27-Pad2): track 0.00 -> 14.8 mm
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