File: MacroBoard/MacroBoard.kicad_sch (KiCad schematic)
At the start: 100 parts, among them J1 USB_C_Receptacle_USB2.0, SW1 SW_Push, U1 AT90USB1286-AU, Y1 Crystal_GND24_Small

Commit message: finished
Parts:
- removed F1: 500mA, Fuse:Fuse_1206_3216Metric, symbol Device:Polyfuse_Small
- removed FB1: 600R, josh-passives-smt:Ferrite_Bead_0603, symbol pcb-rescue:Ferrite_Bead_Small-Device
- removed J1: USB_C_Receptacle_USB2.0, Connector_USB:USB_C_Receptacle_HRO_TYPE-C-31-M-12, symbol pcb-rescue:USB_C_Receptacle_USB2.0-Connector
- added D41: SMF9.0CA, Diode_SMD:D_SOD-123, symbol Device:D_TVS
- added D42, D43: 1.25V@150mA, led:D_SOD-123, symbol led:D_Small
- added F1: ASMD1206-150, Fuse:Fuse_0603_1608Metric_Pad1.05x0.95mm_HandSolder, symbol Device:Polyfuse
- added J1: TYPE-C-31-M12_13, acheron_Connectors:TYPE-C-31-M-12, symbol Unified-Daughterboard-rescue:TYPE-C-31-M12_13-acheronSymbols
- added L1: 60R@100MHz, Inductor_SMD:L_1206_3216Metric, symbol Unified-Daughterboard-rescue:L_Core_Ferrite-Device
- added SW2, SW3: RotaryEncoder_Switch, led:RotaryEncoder_EC11E-Switch, symbol Device:RotaryEncoder_Switch
- added U2: TPD4E05U06DQAR, acheron_Components:USON-10_2.5x1.0mm_P0.5mm, symbol Unified-Daughterboard-rescue:TPD4E05U06DQAR-acheronSymbols
- R1, R2: value 5K1 -> 5.1k; footprint Resistor_SMD:R_0805_2012Metric -> Resistor_SMD:R_0402_1005Metric_Pad0.72x0.64mm_HandSolder; Package (none) -> R0603
- SW1: footprint random-keyboard-parts:SKQG-1155865 -> led:switch_without_switch
Connections:
- net D+ is gone; now on net DA+: R4.2
- net D- is gone; now on net DA-: R3.2
- net GND: now also L1.1, SW2.C, SW3.C; no longer C1.2, C10.2, C11.2, C12.2, C13.2, C14.2, C15.2, C16.2, C17.2, C18.2, C19.2, C20.2, C21.2, C22.2, C23.2, C24.2, C25.2, C26.2, C27.2, C28.2, C9.2, D21.2 (VSS), D22.2 (VSS), D23.2 (VSS), D24.2 (VSS), D25.2 (VSS), D26.2 (VSS), D27.2 (VSS), D28.2 (VSS), D29.2 (VSS), D30.2 (VSS), D31.2 (VSS), D32.2 (VSS), D33.2 (VSS), D34.2 (VSS), D35.2 (VSS), D36.2 (VSS), D37.2 (VSS), D38.2 (VSS), D39.2 (VSS), D40.2 (VSS), R1.1, R2.1
- net ROW0: now also D42.1 (K)
- net ROW1: now also D43.1 (K)
- net VCC: now also D41.2 (A2), F1.2; no longer C1.1
- net GNDREF: now reaches R1.2
- net GNDREF: now also C1.2, C10.2, C11.2, C12.2, C13.2, C14.2, C15.2, C16.2, C17.2, C18.2, C19.2, C20.2, C21.2, C22.2, C23.2, C24.2, C25.2, C26.2, C27.2, C28.2, C9.2, D21.2 (VSS), D22.2 (VSS), D23.2 (VSS), D24.2 (VSS), D25.2 (VSS), D26.2 (VSS), D27.2 (VSS), D28.2 (VSS), D29.2 (VSS), D30.2 (VSS), D31.2 (VSS), D32.2 (VSS), D33.2 (VSS), D34.2 (VSS), D35.2 (VSS), D36.2 (VSS), D37.2 (VSS), D38.2 (VSS), D39.2 (VSS), D40.2 (VSS), R2.2, D41.1 (A1), J1.A1 (GND), J1.B1 (GND), L1.2, U2.3 (GND), U2.8 (GND)
- net DA-: now reaches R3.1, U1.4 (D-)
- net DA-: now also J1.A7 (D-), J1.B7 (D-), U2.2 (IO2), U2.5 (D2-), U2.6 (NC), U2.9 (NC)
- net ROT_2A: now reaches U1.12 (PB2)
- net ROT_2A: now also SW3.A
- net ROT_2B: now reaches U1.13 (PB3)
- net ROT_2B: now also SW3.B
- net ROT_1A: now reaches U1.14 (PB4)
- net ROT_1A: now also SW2.A
- net ROT_1B: now reaches U1.15 (PB5)
- net ROT_1B: now also SW2.B
- net COL5: now reaches U1.38 (PC3)
- net DA+: now reaches R4.1, U1.5 (D+)
- net DA+: now also J1.A6 (D+), J1.B6 (D+), U2.1 (IO1), U2.10 (NC), U2.4 (D2+), U2.7 (NC)
- new net: D43.2 (A), SW3.S1
- new net: D42.2 (A), SW2.S1
- new net: J1.A5 (CC1), R1.1
- new net: J1.B5 (CC2), R2.1
- new net: SW2.S2, SW3.S2
- new net GNDPWR: J1.S (SHIELD)
- new net VBUS: C1.1, F1.1, J1.A4 (VBUS), J1.B4 (VBUS)
- no-connect marks 0 -> 2
Other:
- note added: "Connector and shield"
- note added: "ESD"
- moved on the sheet: C10, C11, C12, C13, C14, C15, C16, C17, C18, C19, C20, C21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

Commit message: cleanup
Parts:
- added H1: (no value), symbol Mechanical:MountingHole
- added H2, H3, H4, H5, H6, H7, H8, H9: MountingHole, symbol Mechanical:MountingHole
- added R7: (no value), Resistor_SMD:R_0402_1005Metric_Pad0.72x0.64mm_HandSolder, symbol Device:R_Small
Connections:
- net VCC is gone; now on net +5V: D41.2 (A2), F1.2
- net VBUS: now also R7.2; no longer J1.A4 (VBUS), J1.B4 (VBUS)
- new net: J1.A4 (VBUS), J1.B4 (VBUS), R7.1

Commit message: generate final Gerber
Parts:
- added Q1: 2N7002, Package_TO_SOT_SMD:SOT-23, symbol Transistor_FET:2N7002
- added R10: 46, Resistor_SMD:R_0805_2012Metric, symbol Device:R_Small
- added R8, R9: 10k, Resistor_SMD:R_0805_2012Metric, symbol Device:R_Small
- H1: value (none) -> MountingHole; footprint (none) -> MountingHole:MountingHole_2.2mm_M2
- H2, H3, H4, H5, H6, H7, H8, H9: footprint (none) -> MountingHole:MountingHole_2.2mm_M2
- R7: value (none) -> 60; footprint Resistor_SMD:R_0402_1005Metric_Pad0.72x0.64mm_HandSolder -> Resistor_SMD:R_0805_2012Metric_Pad1.20x1.40mm_HandSolder; Package R0603 -> R0505
Connections:
- net +5V: now also R7.2; no longer C10.1, C11.1, C12.1, C13.1, C14.1, C15.1, C16.1, C17.1, C18.1, C19.1, C20.1, C21.1, C22.1, C23.1, C24.1, C25.1, C26.1, C27.1, C28.1, C9.1, D21.4 (VDD), D22.4 (VDD), D23.4 (VDD), D24.4 (VDD), D25.4 (VDD), D26.4 (VDD), D27.4 (VDD), D28.4 (VDD), D29.4 (VDD), D30.4 (VDD), D31.4 (VDD), D32.4 (VDD), D33.4 (VDD), D34.4 (VDD), D35.4 (VDD), D36.4 (VDD), D37.4 (VDD), D38.4 (VDD), D39.4 (VDD), D40.4 (VDD), D41.2 (A2), F1.2
- net GNDREF: now also R9.1
- net VBUS: now also J1.A4 (VBUS), J1.B4 (VBUS); no longer R7.2
- net at U1.42 (PC7): now also R8.2
- new net: Q1.1 (G), R8.1, R9.2
- new net: Q1.2 (S), R10.1
- new net Power: D41.2 (A2), F1.2, R10.2, R7.1
- new net Power_LED: C10.1, C11.1, C12.1, C13.1, C14.1, C15.1, C16.1, C17.1, C18.1, C19.1, C20.1, C21.1, C22.1, C23.1, C24.1, C25.1, C26.1, C27.1, C28.1, C9.1, D21.4 (VDD), D22.4 (VDD), D23.4 (VDD), D24.4 (VDD), D25.4 (VDD), D26.4 (VDD), D27.4 (VDD), D28.4 (VDD), D29.4 (VDD), D30.4 (VDD), D31.4 (VDD), D32.4 (VDD), D33.4 (VDD), D34.4 (VDD), D35.4 (VDD), D36.4 (VDD), D37.4 (VDD), D38.4 (VDD), D39.4 (VDD), D40.4 (VDD), Q1.3 (D)

Commit message: fixed lights
Parts:
- D21, D22, D23, D24, D25, D26, D27, D28, D29, D30, D31, D32, D33, D34, D35, D36, D37, D38, D39, D40: symbol LED:SK6812MINI -> randomSymbols:SK6812MINI-E
Connections:
- net COL0: now also U1.34 (PE1); no longer U1.33 (PE0)
- net COL1: now also U1.35 (PC0); no longer U1.34 (PE1)
- net COL2: now also U1.36 (PC1); no longer U1.35 (PC0)
- net COL3: now also U1.37 (PC2); no longer U1.36 (PC1)
- net COL4: now also U1.38 (PC3); no longer U1.37 (PC2)
- net COL5: now also SW2.S2, SW3.S2, U1.13 (PB3); no longer U1.38 (PC3)
- net DataIN: now also D21.4 (DIN), U1.33 (PE0); no longer D21.3 (DIN)
- net DataOUT: now also D40.2 (DOUT); no longer D40.1 (DOUT)
- net GNDREF: now also D21.3 (GND), D22.3 (GND), D23.3 (GND), D24.3 (GND), D25.3 (GND), D26.3 (GND), D27.3 (GND), D28.3 (GND), D29.3 (GND), D30.3 (GND), D31.3 (GND), D32.3 (GND), D33.3 (GND), D34.3 (GND), D35.3 (GND), D36.3 (GND), D37.3 (GND), D38.3 (GND), D39.3 (GND), D40.3 (GND); no longer D21.2 (VSS), D22.2 (VSS), D23.2 (VSS), D24.2 (VSS), D25.2 (VSS), D26.2 (VSS), D27.2 (VSS), D28.2 (VSS), D29.2 (VSS), D30.2 (VSS), D31.2 (VSS), D32.2 (VSS), D33.2 (VSS), D34.2 (VSS), D35.2 (VSS), D36.2 (VSS), D37.2 (VSS), D38.2 (VSS), D39.2 (VSS), D40.2 (VSS)
- net Power_LED: now also D21.1 (VDD), D22.1 (VDD), D23.1 (VDD), D24.1 (VDD), D25.1 (VDD), D26.1 (VDD), D27.1 (VDD), D28.1 (VDD), D29.1 (VDD), D30.1 (VDD), D31.1 (VDD), D32.1 (VDD), D33.1 (VDD), D34.1 (VDD), D35.1 (VDD), D36.1 (VDD), D37.1 (VDD), D38.1 (VDD), D39.1 (VDD), D40.1 (VDD); no longer D21.4 (VDD), D22.4 (VDD), D23.4 (VDD), D24.4 (VDD), D25.4 (VDD), D26.4 (VDD), D27.4 (VDD), D28.4 (VDD), D29.4 (VDD), D30.4 (VDD), D31.4 (VDD), D32.4 (VDD), D33.4 (VDD), D34.4 (VDD), D35.4 (VDD), D36.4 (VDD), D37.4 (VDD), D38.4 (VDD), D39.4 (VDD), D40.4 (VDD)
- net ROT_2A: now also U1.11 (PB1); no longer U1.12 (PB2)
- net ROT_2B: now also U1.12 (PB2); no longer U1.13 (PB3)
- new net: D25.2 (DOUT), D29.4 (DIN)
- new net: D21.2 (DOUT), D25.4 (DIN)
- new net: D22.2 (DOUT), D26.4 (DIN)
- new net: D22.4 (DIN), D37.2 (DOUT)
- new net: D27.2 (DOUT), D31.4 (DIN)
- new net: D23.2 (DOUT), D27.4 (DIN)
- new net: D36.2 (DOUT), D40.4 (DIN)
- new net: D32.2 (DOUT), D36.4 (DIN)
- new net: D26.2 (DOUT), D30.4 (DIN)
- new net: D28.2 (DOUT), D32.4 (DIN)
- new net: D24.2 (DOUT), D28.4 (DIN)
- new net: D23.4 (DIN), D38.2 (DOUT)
- new net: D34.2 (DOUT), D38.4 (DIN)
- new net: D33.2 (DOUT), D37.4 (DIN)
- new net: D29.2 (DOUT), D33.4 (DIN)
- new net: D35.2 (DOUT), D39.4 (DIN)
- new net: D31.2 (DOUT), D35.4 (DIN)
- new net: D30.2 (DOUT), D34.4 (DIN)
- new net: D24.4 (DIN), D39.2 (DOUT)
